Commit message: 1. changed mujoco collision check from dynamic to predefined; 2. limited some joint ranges. This works with z-only jumping

File: urdf/jumping_robot_ry.urdf (robot description, URDF)
Before this commit: robot jumping_robot_ry, 14 links, 13 joints
Joints:
- joint ankle_left_y: limit lower=0.0 upper=1.7 effort=280 velocity=60.62 -> lower=-0.4 upper=0.7 effort=280 velocity=12.62
- joint ankle_right_y: limit lower=-0.4 upper=1.4 effort=280 velocity=60.62 -> lower=-0.4 upper=0.7 effort=280 velocity=12.62
- joint knee_left: limit lower=-2.4 upper=1.14 effort=280 velocity=60.62 -> lower=-2.4 upper=0.0 effort=280 velocity=60.62
